File: hardware/V2_board-ecar/V2_board-ecar.kicad_sch (KiCad schematic)
At the start: 99 parts, among them IC1 ATMEGA8A-P, J1 2x BATT IN, J10 24V, J11 18V, J12 5V, J13 Analog-in-2 0-5V, J14 IGBT, J15 Analog-in-3 - 30to5 (batt), J17 2x Switch (to 5V), J18 Relay contacts, J19 2x 5V, J2 ST 2x GND, J20 ADC Battery, J21 ADC reserve, J22 ADC Gas-pedal, J23 2x 24V filtered, J24 GND-supp, Diode, Mosfet (fan), J3 2x 24V filtered, J4 ST 2x GND, J5 PWM-Signal, J6 LED ~3,2V 20mA, J7 Gas Pedal, J8 Gate, J9 BATT, K1 LEG-5, P1 ISP, Q1 BC547, Q2 IRFZ24N, Q3 BC547, U1 LM7818CT, U2 LM2576T-5, U3 TC429

Commit message: pcb: re-arrange schematic, fix track widths
Other:
- note added: "Filter out 50V peaks on battery voltage each pwm cycle"
- note added: "ISP Programmer connector"
- note added: "Power Terminals"
- note removed: "Filter 50V peaks on battery voltage each pwm cycle"
- moved on the sheet: BZ1, C1, C10, C11, C12, C13, C14, C15, C16, C17, C18, C19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

Commit message: pcb: Fix footprints, add pcb2gcode conf from ihc-control_pcb project
Parts:
- BZ1: footprint Buzzer_Beeper:MagneticBuzzer_ProSignal_ABT-410-RC -> Buzzer_Beeper:Buzzer_TDK_PS1240P02BT_D12.2mm_H6.5mm
Changed lines of the file:
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@@
 			)
 		)
-		(property "Footprint" "Buzzer_Beeper:MagneticBuzzer_ProSignal_ABT-410-RC"
+		(property "Footprint" "Buzzer_Beeper:Buzzer_TDK_PS1240P02BT_D12.2mm_H6.5mm"
 			(at 297.815 215.9 90)
 			(effects

Commit message: pcb: adjust silk, version milled (track missing)
Other:
- note added: "gas pedal measurements: 5V-GND: ~1k Ohm when released, ~1k when pressed OUT-GND and OUT-5V: moves between 0.9k to 1.7k"
- note removed: "TODO: measure gas pedal voltage-drivider resistance -> choose R high enough"
Changed lines of the file:
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@@
 		)
 	)
-	(text "TODO: measure gas pedal voltage-drivider resistance\n-> choose R high enough"
+	(text "gas pedal measurements: \n5V-GND: ~1k Ohm when released, ~1k when pressed\nOUT-GND and OUT-5V: moves between 0.9k to 1.7k "
 		(exclude_from_sim no)
-		(at 202.438 54.356 0)
+		(at 197.104 82.804 0)
 		(effects
 			(font

Commit message: pcb: Fix missing tracks, Annotate schematic and layout
Parts:
- D3: value TVS 26V (starts 31V) -> TVS 28V (starts 31V)
- F1: value 500mA -> slow, max 4A
- F3: value 500mA -> (H7 24V 70W) -> 3A
- J14: value IGBT -> IGBT [GND, Gate]
- J18: value Relay contacts -> Relay contacts [NO, COM, NC]
- J24: value GND-supp, Diode, Mosfet (fan) -> Fan [GND-supp, Diode, Mosfet]
- J6: value LED ~3,2V 20mA -> LED 3,2V 20mA [-, +]
- R16: value 150k -> 100k
- R17: value 30k -> 22k
- R9: value 12k -> 12k (15k used)
Other:
- note added: "24V Supply (voltage filter)"
- note added: "Atmega-8 Microcontroller"
- note added: "Input voltage range: 20V to 35V"
- note removed: "24V Supply voltage filter"
- title: (none) -> New version of PCB controlling an electric kart
- moved on the sheet: C1, C11, C12, C13, C14, C15, C16, C19, C2, C3, C5, C6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
